Commit message: Get real robot working

File: description/lidar.xacro (robot description, xacro)
@@ -1,15 +1,22 @@
 <?xml version="1.0"?>
-<robot xmlns:xacro="http://www.ros.org/wiki/xacro">
+<robot xmlns:xacro="http://www.ros.org/wiki/xacro" >
     <joint name="laser_joint" type="fixed">
         <parent link="chassis"/>
         <child link="laser_frame"/>
-        <origin xyz="0.2 0 0.175" rpy="0 0 0"/>
+        <origin xyz="0.094 0 0.1326" rpy="0 0 0"/>
     </joint>
     <link name="laser_frame">
         <visual>
             <geometry>
-                <cylinder radius="0.05" length="0.04"/>
+                <cylinder radius="0.04" length="0.034"/>
             </geometry>
-            <material name="red"/>
+            <material name="black"/>
+        </visual>
+        <visual>
+            <origin xyz="0 0 -0.0248"/>
+            <geometry>
+                <cylinder radius="0.01" length="0.0156"/>
+            </geometry>
+            <material name="black"/>
         </visual>
         <collision>
@@ -18,13 +25,13 @@
             </geometry>
         </collision>
-        <xacro:inertial_cylinder mass="0.1" radius="0.05" length="0.04">
+        <xacro:inertial_cylinder mass="0.2" length="0.04" radius="0.05">
             <origin xyz="0 0 0" rpy="0 0 0"/>
         </xacro:inertial_cylinder>
     </link>
     <gazebo reference="laser_frame">
-        <material>Gazebo/Red</material>
+        <material>Gazebo/Black</material>
         <sensor name="laser" type="ray">
             <pose> 0 0 0 0 0 0 </pose>
-            <visualize>true</visualize>
+            <visualize>false</visualize>
             <update_rate>10</update_rate>
             <ray>

File: description/robot.urdf.xacro (robot description, xacro)
@@ -1,8 +1,8 @@
 <?xml version="1.0"?>
 <robot xmlns:xacro="http://www.ros.org/wiki/xacro"  name="robot">
-    <xacro:include filename="lidar_real.xacro" />
-    <xacro:include filename="robot_hardware.xacro" />
-    <!-- <xacro:include filename="robot_core.xacro" />
-    <xacro:include filename="lidar.xacro" /> -->
+    <!-- <xacro:include filename="lidar_real.xacro" />
+    <xacro:include filename="robot_hardware.xacro" /> -->
+    <xacro:include filename="robot_core.xacro" />
+    <xacro:include filename="lidar.xacro" />
     <!-- <xacro:include filename="gazebo_control.xacro" /> -->
     <xacro:include filename="ros2_control.xacro" />

File: description/robot_core.xacro (robot description, xacro)
@@ -1,49 +1,63 @@
 <?xml version="1.0"?>
 <robot xmlns:xacro="http://www.ros.org/wiki/xacro" >
-    <xacro:include filename="inertial_macros.xacro" />
+    <xacro:include filename="inertial_macros.xacro"/>
+    <xacro:property name="chassis_length" value="0.25"/>
+    <xacro:property name="chassis_width" value="0.15"/>
+    <xacro:property name="chassis_height" value="0.1"/>
+    <xacro:property name="chassis_mass" value="1.85"/>
+    <xacro:property name="wheel_radius" value="0.0335"/>
+    <xacro:property name="wheel_thickness" value="0.026"/>
+    <xacro:property name="wheel_mass" value="0.05"/>
+    <xacro:property name="wheel_offset_x" value="0.21"/>
+    <xacro:property name="wheel_offset_y" value="0.094"/>
+    <xacro:property name="wheel_offset_z" value="0.02"/>
+    <xacro:property name="caster_wheel_radius" value="0.008"/>
+    <xacro:property name="caster_wheel_mass" value="0.01"/>
+    <xacro:property name="caster_wheel_offset_x" value="0.03"/>
+    <xacro:property name="caster_wheel_offset_z" value="${-wheel_offset_z - wheel_radius + caster_wheel_radius}"/>
     <material name="white">
         <color rgba="1 1 1 1" />
     </material>
     <material name="orange">
-        <color rgba="1 0.3 0.1 1" />
+        <color rgba="1 0.3 0.1 1"/>
     </material>
     <material name="blue">
-        <color rgba="0.2 0.2 1 1" />
+        <color rgba="0.2 0.2 1 1"/>
     </material>
     <material name="black">
-        <color rgba="0 0 0 1" />
+        <color rgba="0 0 0 1"/>
     </material>
     <material name="red">
-        <color rgba="1 0 0 1" />
+        <color rgba="1 0 0 1"/>
     </material>
     <!-- BASE LINK -->
     <link name="base_link">
     </link>
-    <!-- CHASSIC LINK -->
+    <!-- CHASSIS LINK -->
     <joint name="chassis_joint" type="fixed">
         <parent link="base_link"/>
         <child link="chassis"/>
-        <origin xyz="-0.1 0 0"/>
+        <origin xyz="${-wheel_offset_x} 0 ${wheel_offset_z}"/>
     </joint>
     <link name="chassis">
         <visual>
-            <origin xyz="0.15 0 0.075"/>
+            <origin xyz="${chassis_length/2} 0 ${chassis_height/2}"/>
             <geometry>
-                <box size="0.3 0.3 0.15"/>
+                <box size="${chassis_length} ${chassis_width} ${chassis_height}"/>
             </geometry>
-            <material name="white"/>
+            <material name="orange"/>
         </visual>
         <collision>
-            <origin xyz="0.15 0 0.075"/>
+            <origin xyz="${chassis_length/2} 0 ${chassis_height/2}"/>
             <geometry>
-                <box size="0.3 0.3 0.15"/>
+                <box size="${chassis_length} ${chassis_width} ${chassis_height}"/>
             </geometry>
         </collision>
-        <xacro:inertial_box mass="0.5" x="0.3" y="0.3" z="0.15">
-            <origin xyz="0.15 0 0.075" rpy="0 0 0"/>
+        <xacro:inertial_box mass="${chassis_mass}" x="${chassis_length}" y="${chassis_width}" z="${chassis_height}">
+            <origin xyz="${chassis_length/2} 0 ${chassis_height/2}" rpy="0 0 0"/>
         </xacro:inertial_box>
     </link>
     <gazebo reference="chassis">
-        <material>Gazebo/White</material>
+        <material>Gazebo/Orange</material>
     </gazebo>
     <!-- LEFT WHEEL LINK -->
@@ -51,11 +65,11 @@
         <parent link="base_link"/>
         <child link="left_wheel"/>
-        <origin xyz="0 0.175 0" rpy="-${pi/2} 0 0"/>
-        <axis xyz="0 0 1"/>
+        <origin xyz="0 ${wheel_offset_y} 0" rpy="-${pi/2} 0 0" />
+        <axis xyz="0 0 -1"/>
     </joint>
     <link name="left_wheel">
         <visual>
             <geometry>
-                <cylinder radius="0.05" length="0.04"/>
+                <cylinder radius="${wheel_radius}" length="${wheel_thickness}"/>
             </geometry>
             <material name="blue"/>
@@ -63,8 +77,8 @@
         <collision>
             <geometry>
-                <cylinder radius="0.05" length="0.04"/>
+                <sphere radius="${wheel_radius}"/>
             </geometry>
         </collision>
-        <xacro:inertial_cylinder mass="0.1" radius="0.05" length="0.04">
+        <xacro:inertial_cylinder mass="${wheel_mass}" length="${wheel_thickness}" radius="${wheel_radius}">
             <origin xyz="0 0 0" rpy="0 0 0"/>
         </xacro:inertial_cylinder>
@@ -73,15 +87,15 @@
         <material>Gazebo/Blue</material>
     </gazebo>
-        <!-- RIGHT WHEEL LINK -->
+    <!-- RIGHT WHEEL LINK -->
     <joint name="right_wheel_joint" type="continuous">
         <parent link="base_link"/>
         <child link="right_wheel"/>
-        <origin xyz="0 -0.175 0" rpy="${pi/2} 0 0"/>
-        <axis xyz="0 0 -1"/>
+        <origin xyz="0 ${-wheel_offset_y} 0" rpy="${pi/2} 0 0" />
+        <axis xyz="0 0 1"/>
     </joint>
     <link name="right_wheel">
         <visual>
             <geometry>
-                <cylinder radius="0.05" length="0.04"/>
+                <cylinder radius="${wheel_radius}" length="${wheel_thickness}"/>
             </geometry>
             <material name="blue"/>
@@ -89,8 +103,8 @@
         <collision>
             <geometry>
-                <cylinder radius="0.05" length="0.04"/>
+                <sphere radius="${wheel_radius}"/>
             </geometry>
         </collision>
-        <xacro:inertial_cylinder mass="0.1" radius="0.05" length="0.04">
+        <xacro:inertial_cylinder mass="${wheel_mass}" length="${wheel_thickness}" radius="${wheel_radius}">
             <origin xyz="0 0 0" rpy="0 0 0"/>
         </xacro:inertial_cylinder>
@@ -103,10 +117,24 @@
         <parent link="chassis"/>
         <child link="caster_wheel"/>
-        <origin xyz="0.24 0 0"/>
+        <origin xyz="${caster_wheel_offset_x} 0 ${caster_wheel_offset_z}"/>
     </joint>
     <link name="caster_wheel">
         <visual>
             <geometry>
-                <sphere radius="0.05"/>
+                <sphere radius="${caster_wheel_radius}"/>
+            </geometry>
+            <material name="white"/>
+        </visual>
+        <visual>
+            <origin xyz="0 0.012 0.02275"/>
+            <geometry>
+                <cylinder radius="0.003" length="0.0455"/>
+            </geometry>
+            <material name="black"/>
+        </visual>
+                <visual>
+            <origin xyz="0 -0.012 0.02275"/>
+            <geometry>
+                <cylinder radius="0.003" length="0.0455"/>
             </geometry>
             <material name="black"/>
@@ -114,13 +142,13 @@
         <collision>
             <geometry>
-                <sphere radius="0.05"/>
+                <sphere radius="${caster_wheel_radius}"/>
             </geometry>
         </collision>
-        <xacro:inertial_sphere mass="0.1" radius="0.05">
+        <xacro:inertial_sphere mass="${caster_wheel_mass}" radius="${caster_wheel_radius}">
             <origin xyz="0 0 0" rpy="0 0 0"/>
         </xacro:inertial_sphere>
     </link>
     <gazebo reference="caster_wheel">
-        <material>Gazebo/Black</material>
+        <material>Gazebo/White</material>
         <mu1 value="0.001"/>
         <mu2 value="0.001"/>

File: description/robot_hardware.xacro (robot description, xacro)
@@ -20,23 +20,21 @@
     <visual>
       <origin
-        xyz="0 0 0"
-        rpy="0 0 0" />
-      <geometry>
-        <mesh
-          filename="file:$(find my_mobrob)/meshes/chassis.STL" />
-      </geometry>
-      <material
-        name="">
-        <color
-          rgba="0.79216 0.81961 0.93333 1" />
-      </material>
-    </visual>
-    <collision>
-      <origin
-        xyz="0 0 0"
-        rpy="0 0 0" />
-      <geometry>
-        <mesh
-          filename="file:$(find my_mobrob)/meshes/chassis.STL" />
+        xyz="0.125 0 0.025"
+        rpy="0 0 0" />
+      <geometry>
+        <box size="0.25 0.15 0.05"/>
+      </geometry>
+      <material
+        name="">
+        <color
+          rgba="0.79216 0.81961 0.93333 1" />
+      </material>
+    </visual>
+    <collision>
+      <origin
+        xyz="0.125 0 0.025"
+        rpy="0 0 0" />
+      <geometry>
+        <box size="0.25 0.15 0.05"/>
       </geometry>
     </collision>
@@ -74,20 +72,18 @@
         rpy="0 0 0" />
       <geometry>
-        <mesh
-          filename="file:$(find my_mobrob)/meshes/caster_wheel.STL" />
-      </geometry>
-      <material
-        name="">
-        <color
-          rgba="0.79216 0.81961 0.93333 1" />
-      </material>
-    </visual>
-    <collision>
-      <origin
-        xyz="0 0 0"
-        rpy="0 0 0" />
-      <geometry>
-        <mesh
-          filename="file:$(find my_mobrob)/meshes/caster_wheel.STL" />
+          <sphere radius="0.007"/>
+      </geometry>
+      <material
+        name="">
+        <color
+          rgba="0.79216 0.81961 0.93333 1" />
+      </material>
+    </visual>
+    <collision>
+      <origin
+        xyz="0 0 0"
+        rpy="0 0 0" />
+      <geometry>
+          <sphere radius="0.007"/>
       </geometry>
     </collision>
@@ -136,5 +132,5 @@
     <collision>
       <origin
-        xyz="0 0 0"
+        xyz="0 8.6E-03 0"
         rpy="0 0 0" />
       <geometry>

Commit message: update_urdf

File: description/lidar.xacro (robot description, xacro)
@@ -2,7 +2,7 @@
 <robot xmlns:xacro="http://www.ros.org/wiki/xacro" >
     <joint name="laser_joint" type="fixed">
-        <parent link="chassis"/>
+        <parent link="base_link"/>
         <child link="laser_frame"/>
-        <origin xyz="0.094 0 0.1326" rpy="0 0 0"/>
+        <origin xyz="-0.116 0 0.1526" rpy="0 0 0"/>
     </joint>
     <link name="laser_frame">

File: description/robot_core.xacro (robot description, xacro)
@@ -34,5 +34,5 @@
     <link name="base_link">
     </link>
-        <!-- BASE_FOOTPRINT LINK -->
+    <!-- BASE_FOOTPRINT LINK -->
     <joint name="base_footprint_joint" type="fixed">
         <parent link="base_link"/>
@@ -73,9 +73,10 @@
         <parent link="base_link"/>
         <child link="left_wheel"/>
-        <origin xyz="0 ${wheel_offset_y} 0" rpy="-${pi/2} 0 0" />
-        <axis xyz="0 0 -1"/>
+        <origin xyz="0 ${wheel_offset_y} 0" rpy="0 0 0" />
+        <axis xyz="0 1 0"/>
     </joint>
     <link name="left_wheel">
         <visual>
+            <origin xyz="0 0 0" rpy="${pi/2} 0 0"/>
             <geometry>
                 <cylinder radius="${wheel_radius}" length="${wheel_thickness}"/>
@@ -84,6 +85,7 @@
         </visual>
         <collision>
+            <origin xyz="0 0 0" rpy="${pi/2} 0 0"/>
             <geometry>
-                <sphere radius="${wheel_radius}"/>
+                <cylinder radius="${wheel_radius}" length="${wheel_thickness}"/>
             </geometry>
         </collision>
@@ -99,9 +101,10 @@
         <parent link="base_link"/>
         <child link="right_wheel"/>
-        <origin xyz="0 ${-wheel_offset_y} 0" rpy="${pi/2} 0 0" />
-        <axis xyz="0 0 1"/>
+        <origin xyz="0 ${-wheel_offset_y} 0" rpy="0 0 0" />
+        <axis xyz="0 1 0"/>
     </joint>
     <link name="right_wheel">
         <visual>
+            <origin xyz="0 0 0" rpy="${pi/2} 0 0"/>
             <geometry>
                 <cylinder radius="${wheel_radius}" length="${wheel_thickness}"/>
@@ -110,6 +113,7 @@
         </visual>
         <collision>
+            <origin xyz="0 0 0" rpy="${pi/2} 0 0"/>
             <geometry>
-                <sphere radius="${wheel_radius}"/>
+                <cylinder radius="${wheel_radius}" length="${wheel_thickness}"/>
             </geometry>
         </collision>
